File: tcan.kicad_sch (KiCad schematic)
At the start: 7 parts, among them J12 Conn_01x02_Socket, J13 Conn_01x02_Socket, SW5 SW_DPDT_x2, U5 TCAN3414DRBR

Commit message: サーボときんていをつけ忘れていたので回路図に追加(部品配置に悩んでる
Parts:
- renumbered C17 to C19, C18 to C20, J12 to J15, J13 to J16, SW5 to SW4
Changed lines of the file:
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@@
 		(dnp no)
 		(fields_autoplaced yes)
-		(property "Reference" "#PWR032"
+		(property "Reference" "#PWR038"
 			(at 104.14 85.09 0)
 			(hide yes)
@@
 			(project "ARSTM2602"
 				(path "/537f457d-9719-41ea-89c7-39afb0f25936/2c046ef4-62ef-4d9d-801e-bfe3df84301b"
-					(reference "#PWR032")
+					(reference "#PWR038")
 					(unit 1)
 				)
@@
 		(in_pos_files yes)
 		(dnp no)
-		(property "Reference" "C18"
+		(property "Reference" "C20"
 			(at 113.792 52.07 0)
 			(show_name no)
@@
 			(project "ARSTM2602"
 				(path "/537f457d-9719-41ea-89c7-39afb0f25936/2c046ef4-62ef-4d9d-801e-bfe3df84301b"
-					(reference "C18")
+					(reference "C20")
 					(unit 1)
 				)
@@
 		(dnp no)
 		(fields_autoplaced yes)
-		(property "Reference" "#PWR033"
+		(property "Reference" "#PWR039"
 			(at 106.68 67.31 0)
 			(hide yes)
@@
 			(project "ARSTM2602"
 				(path "/537f457d-9719-41ea-89c7-39afb0f25936/2c046ef4-62ef-4d9d-801e-bfe3df84301b"
-					(reference "#PWR033")
+					(reference "#PWR039")
 					(unit 1)
 				)
@@
 		(dnp no)
 		(fields_autoplaced yes)
-		(property "Reference" "#PWR031"
+		(property "Reference" "#PWR037"
 			(at 69.85 68.58 0)
 			(hide yes)
@@
 			(project "ARSTM2602"
 				(path "/537f457d-9719-41ea-89c7-39afb0f25936/2c046ef4-62ef-4d9d-801e-bfe3df84301b"
-					(reference "#PWR031")
+					(reference "#PWR037")
 					(unit 1)
 				)
@@
 		(dnp no)
 		(fields_autoplaced yes)
-		(property "Reference" "#PWR034"
+		(property "Reference" "#PWR040"
 			(at 114.3 52.07 0)
 			(hide yes)
@@
 			(project "ARSTM2602"
 				(path "/537f457d-9719-41ea-89c7-39afb0f25936/2c046ef4-62ef-4d9d-801e-bfe3df84301b"
-					(reference "#PWR034")
+					(reference "#PWR040")
 					(unit 1)
 				)
@@
 		(in_pos_files yes)
 		(dnp no)
-		(property "Reference" "J12"
+		(property "Reference" "J15"
 			(at 87.63 86.3599 0)
 			(show_name no)
@@
 			(project "ARSTM2602"
 				(path "/537f457d-9719-41ea-89c7-39afb0f25936/2c046ef4-62ef-4d9d-801e-bfe3df84301b"
-					(reference "J12")
+					(reference "J15")
 					(unit 1)
 				)
@@
 		(dnp no)
 		(fields_autoplaced yes)
-		(property "Reference" "SW5"
+		(property "Reference" "SW4"
 			(at 63.5 74.93 0)
 			(show_name no)
@@
 			(project "ARSTM2602"
 				(path "/537f457d-9719-41ea-89c7-39afb0f25936/2c046ef4-62ef-4d9d-801e-bfe3df84301b"
-					(reference "SW5")
+					(reference "SW4")
 					(unit 1)
 				)
@@
 		(in_pos_files yes)
 		(dnp no)
-		(property "Reference" "J13"
+		(property "Reference" "J16"
 			(at 109.22 86.3599 0)
 			(show_name no)
@@
 			(project "ARSTM2602"
 				(path "/537f457d-9719-41ea-89c7-39afb0f25936/2c046ef4-62ef-4d9d-801e-bfe3df84301b"
-					(reference "J13")
+					(reference "J16")
 					(unit 1)
 				)
@@
 		(in_pos_files yes)
 		(dnp no)
-		(property "Reference" "C17"
+		(property "Reference" "C19"
 			(at 103.378 52.324 0)
 			(show_name no)
@@
 			(project "ARSTM2602"
 				(path "/537f457d-9719-41ea-89c7-39afb0f25936/2c046ef4-62ef-4d9d-801e-bfe3df84301b"
-					(reference "C17")
-					(unit 1)
-				)
+					(reference "C19")
+					(unit 1)
+				)
