File: ARSTM2602.kicad_pcb (KiCad board)
At the start: 2 copper layers, 100 x 100 mm, 113 parts, among them J1 Conn_01x03_Pin, J10 Conn_01x02_Socket, J11 Conn_01x02_Socket, J12 Conn_ST_STDC14, J13 USB_C_Receptacle_USB2.0_14P, J14 Conn_01x02_Socket, J15 Conn_01x02_Socket, J16 Conn_01x02_Socket, J17 USB_C_Receptacle_USB2.0_14P, J18 Conn_01x02_Socket, J19 Conn_01x02_Socket, J2 Conn_01x03_Pin, J20 Conn_01x02_Socket, J21 Conn_01x02_Socket, J22 Conn_01x02_Socket, J23 Conn_01x02_Socket, J3 Conn_01x03_Pin, J4 Conn_01x03_Pin, J5 Conn_01x03_Pin, J6 Conn_01x03_Pin, J7 Conn_01x03_Pin, J8 Conn_01x03_Pin, J9 Conn_01x02_Socket, Q1 Q_NMOS_GSD, Q2 Q_NMOS_GSD, Q3 Q_NMOS_GSD, Q4 Q_NMOS_GSD, Q5 Q_NMOS_GSD, SW1 SW_Push, SW2 SW_Push, SW3 SW_Push, SW4 SW_DPDT_x2, SW5 SW_Push, SW6 SW_Push, U1 STM32G431RBTx, U10 TLP785, U11 TLP785, U12 TLP785, U2 BD33FC0FP, U3 ESP32-C3-WROOM-02, U4 BD33FC0FP, U5 TCAN3414DRBR, U6 ESP32-C3-WROOM-02, U7 BD33FC0FP, U8 TLP785, U9 TLP785

Commit message: 完成版を上げ忘れていた
Parts:
- moved J12 2.01 mm to (108.4, 68.4)
Routing:
- net GND: track 62.3 -> 45.4 mm, vias 120 -> 185
- net Tim3ch4: track 43.6 -> 47.0 mm
- net Tim3ch3: track 45.3 -> 48.7 mm
- net swdio: track 8.99 -> 11.2 mm
- net swclk: track 8.69 -> 10.9 mm
- net +3.3V: track 138.3 -> 140.5 mm
- net uart2-tx: track 8.12 -> 9.54 mm
- net uart2-rx: track 8.56 -> 9.98 mm
Other:
- board text added: "+ -"
- board text added: "- + emerg sw"
- board text added: "- + emergency sw"
- board text added: "12V-GND-4ch1"
- board text added: "12V-GND-4ch2"
- board text added: "Low-High"
- board text added: "batt USB"
- board text added: "g-33"
- board text added: "motor1"
- board text added: "motor2"
- board text added: "motor3"
- board text added: "motor4"
- board text added: "motor5"
- board text added: "motor6"
- board text added: "servo"
- board text added: "terminating on-off"
